File: lmp91000Breakout/lmp91000Breakout.kicad_pcb (KiCad board)
At the start: 2 copper layers, 36.1 x 26.9 mm, 16 parts, among them J1 Conn_01x01_Male, J2 Conn_01x01_Male, J3 Conn_01x01_Male, U1 LMP91000SDE_NOPB

Commit message: changed stuff
Other:
- board text added: "the project can be found at: github.com/COLVERTYETY/LMP9100BreakoutBoard"
Changed lines of the file:
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@@
   (general
     (thickness 1.6)
-    (drawings 18)
+    (drawings 19)
     (tracks 94)
     (zones 0)
@@
     )
   )
+  (gr_text "the project can be found at:\ngithub.com/COLVERTYETY/LMP9100BreakoutBoard" (at 99.568 76.2) (layer B.SilkS)
+    (effects (font (size 1 0.8) (thickness 0.15)) (justify left mirror))
+  )
   (gr_text 29/09/2021 (at 78.232 80.264) (layer F.Cu)

Commit message: added Qrcode
Parts:
- added G***: LOGO, lmp:qrcode, B.Cu at (82.3, 74.7)
- added REF**: theqrcode, theqrcode, F.Cu at (0.00, 0.00)
Other:
- board text added: "github.com/COLVERTYETY /LMP9100BreakoutBoard"
- board text removed: "the project can be found at: github.com/COLVERTYETY/LMP9100BreakoutBoard"
